File: PCB/kontroler Tomografi/kontroler/kontroler.kicad_sch (KiCad schematic)
At the start: 23 parts, among them J1 In_VCCS, J2 Out_Switch, J3 In_Switch, J4 V_In, U1 AD620, U2 ESP32-S3-DevKitC, U4 L7805

Commit message: PCB kontroler tomografi V2
Parts:
- removed C3: 0.1u, Capacitor_THT:C_Disc_D4.3mm_W1.9mm_P5.00mm, symbol Device:C
- removed J4: V_In, Connector_PinHeader_2.54mm:PinHeader_1x03_P2.54mm_Vertical, symbol Connector_Generic:Conn_01x03
- removed JP1: 100G, Jumper:SolderJumper-2_P1.3mm_Open_RoundedPad1.0x1.5mm, symbol Jumper:SolderJumper_2_Open
- removed JP2: 10G, Jumper:SolderJumper-2_P1.3mm_Open_RoundedPad1.0x1.5mm, symbol Jumper:SolderJumper_2_Open
- removed JP3: 1G, Jumper:SolderJumper-2_P1.3mm_Open_RoundedPad1.0x1.5mm, symbol Jumper:SolderJumper_2_Open
- removed U2: ESP32-S3-DevKitC, PCM_Espressif:ESP32-S3-DevKitC, symbol PCM_Espressif:ESP32-S3-DevKitC
- removed U4: L7805, Package_TO_SOT_THT:TO-220-3_Vertical, symbol Regulator_Linear:L7805
- added J4: Out_Switch, Connector_PinHeader_2.54mm:PinHeader_1x04_P2.54mm_Vertical, symbol Connector_Generic:Conn_01x04
- added J5: Conn_02x04_Odd_Even, Connector_PinHeader_2.54mm:PinHeader_2x04_P2.54mm_Vertical, symbol Connector_Generic:Conn_02x04_Odd_Even
- added R6: 49.4k, Resistor_THT:R_Axial_DIN0207_L6.3mm_D2.5mm_P10.16mm_Horizontal, symbol Device:R
- added R7: R, Resistor_THT:R_Axial_DIN0207_L6.3mm_D2.5mm_P10.16mm_Horizontal, symbol Device:R
- added U4: YAAJ_BluePill, Library:YAAJ_BluePill_1, symbol Libraryy:YAAJ_BluePill
- C2: value 0.33u -> C
- J2: value Out_Switch -> V_In
- R3: value 494 -> 499
- R4: value 4.94k -> 5.94k
Connections:
- net +15V: now also J2.1 (Pin_1); no longer C2.1
- net +3.3V: now also U4.20 (3V3), U4.38 (3V3)
- net +5V: now also U4.18 (5V)
- net +V: now also J4.2 (Pin_2); no longer J2.2 (Pin_2)
- net -15V: now also J2.2 (Pin_2)
- net -V: now also J4.3 (Pin_3); no longer J2.3 (Pin_3)
- net En: now also U4.33 (PB0)
- net GND: now also J2.3 (Pin_3), J4.1 (Pin_1), R7.1, U4.19 (GND), U4.39 (GND), U4.40 (GND); no longer C2.2, J2.1 (Pin_1)
- net Out 9833: now also C2.1; no longer J1.1 (Pin_1)
- net Out ADC: now also U4.25 (PA0)
- net RCLK: now also U4.34 (PB1)
- net SCLR: now also U4.36 (PB11)
- net at R3.1, R4.1, R5.1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: now also R6.1
- net at R5.2: now also J5.4 (Pin_4)
- net at R4.2: now also J5.6 (Pin_6)
- net at U1.8 (Rg): now also J5.1 (Pin_1), J5.3 (Pin_3), J5.5 (Pin_5), J5.7 (Pin_7)
- net at R3.2: now also J5.8 (Pin_8)
- net GPIO10 renamed FSYNC
- net FSYNC: now also U4.29 (PA4)
- net GPIO11 renamed SDATA
- net SDATA: now also U4.32 (PA7)
- net GPIO12 renamed SCLK1
- net SCLK1: now also U4.30 (PA5)
- net SCLK renamed SCLK2
- net SCLK2: now also U4.35 (PB10)
- new net: J5.2 (Pin_2), R6.2
- new net Out HPF: C2.2, J1.1 (Pin_1), R7.2
- new net Out pin ADC: J4.4 (Pin_4), U4.26 (PA1)
- no-connect marks 30 -> 25
Other:
- note added: "High Pass Filter"
- note added: "STM32 Blue Pill"
- note removed: "ESP32-S3-DevKitC"
- note removed: "L7805 IC penstabil tegangan positif"
- moved on the sheet: H1, H2, H3, H4, J2, R1, R2, R3, R4, R5

Commit message: PCB kontroler tomografi V2.1
Parts:
- added J6: V 5V, Connector_PinHeader_2.54mm:PinHeader_1x02_P2.54mm_Vertical, symbol Connector_Generic:Conn_01x02
Connections:
- net +5V: now also J6.2 (Pin_2); no longer J3.1 (Pin_1)
- net +15V renamed +5VA
- net +5VA: now also J3.1 (Pin_1), J6.1 (Pin_1)
- net -15V renamed -5V
Other:
- moved on the sheet: J2, J4
